File: Schematy/STM LQFP32/plytka_glowna.sch (EAGLE design)
At the start: 51 parts, among them IC1 LM1117-3.3V, IC2 74HC595D

Commit message: Płytka główna + listwa z czujnikami
* dodałem listwę z czujnikami
* poprawiłem cewkę przy mikrokontrolerze
* zmieniłem złącze czujników na 1x10
* poprawiłem złącze do modułu bluetooth
Parts:
- J3: device SparkFun-Connectors:M05X2NO_SILK -> SparkFun-Connectors:M10LOCK
Connections:
- net +3V3: now also J3.10; no longer J3.1
- net BLUETOOTH_RX: now also J2.3; no longer J2.4
- net BLUETOOTH_TX: now also J2.4; no longer J2.3
- net GND: now also J3.1; no longer J3.10
- net KTIR_1: now also J3.9; no longer J3.2
- net KTIR_2: now also J3.8; no longer J3.4
- net KTIR_3: now also J3.7; no longer J3.6
- net KTIR_4: now also J3.6; no longer J3.8
- net KTIR_5: now also J3.5; no longer J3.3
- net KTIR_6: now also J3.4; no longer J3.5
- net KTIR_7: now also J3.3; no longer J3.7
- net KTIR_8: now also J3.2; no longer J3.9
- net VDD: no longer L1.2
- net VDDA: now also L1.2
Other:
- moved on the sheet: C3, C4, C5, C6, C7, J3, J4, L1, R12, R13
