File: Schematy/STM LQFP32/płytka główna/plytka_glowna.sch (EAGLE design)
At the start: 51 parts, among them IC1 LM1117-3.3V, IC2 74HC595D, J3 68611014422

Commit message: Płytka gotowa
Parts:
- removed S1, S2: TACTILE-SWITCH-7914G, GeekAmmo:TACTILE-SWITCH-7914G
- added RESET, START: 430186043916, Switches_rev16a:430186043916
- C1, C11, C13, C2: device rcl:CPOL-EU085CS-1AR -> rcl:CPOL-EUUD-4X5,8
- C10, C12, C14, C3, C4, C6, C8, C9: device rcl:C-EU025-024X044 -> rcl:C-EUC0805
- C5, C7: device rcl:CPOL-EU085CS-1AR -> rcl:CPOL-EUSMCA
- L1: device rcl:L-EU0204/7 -> rcl:R-EU_R0805
- R1, R10, R11, R12, R13, R2, R3, R4, R5, R6, R7, R8, R9: device rcl:R-EU_0204/2V -> rcl:R-EU_M0805
- renumbered J1 to PROG, J2 to BLUETOOTH, J4 to BATTERY, J5 to ENG1, J6 to ENG2, U$2 to TB6612FNG
Connections:
- net GND: now also RESET.3, RESET.4, START.3, START.4; no longer S1.3, S1.4, S2.3, S2.4
- net PRZYCISK_START/STOP: now also START.1, START.2; no longer S2.1, S2.2
- net RESET: now also RESET.1, RESET.2; no longer S1.1, S1.2
