File: Schematy/STM LQFP32/płytka główna/plytka_glowna.brd (EAGLE design)
At the start: 150.5 x 72.4 mm, 53 parts, among them IC1 LM1117-3.3V, IC2 74HC595D

Commit message: Poprawione PCB
Routing:
- net GND: track 18.9 -> 27.1 mm
- net LED_WSK_NAL_2: track 50.1 -> 52.0 mm
- net KIERUNEK_1_SILNIK_A: track 27.4 -> 29.1 mm
- net LED_WSK_NAL_1: track 40.0 -> 41.4 mm
- net AKUMULATOR: track 113.8 -> 115.1 mm
- net LED_KTIR_1: track 83.7 -> 84.5 mm
- net KIERUNEK_2_SILNIK_A: vias 2 -> 3
