File: Schematy/STM LQFP32/listwa z czujnikami/listwa_z_czujnikami.brd (EAGLE design)
At the start: 160 x 100 mm, 25 parts, among them J1 68611014122

Commit message: Poprawione PCB
Routing:
- net KTIR_2: vias 1 -> 2
- net GND: vias 8 -> 9
- net +3V3: vias 8 -> 9
Changed lines of the file:
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@@
 <hole x="55.61" y="4" drill="2"/>
 <hole x="80.65" y="4" drill="2"/>
-<hole x="80.72" y="9" drill="2"/>
-<hole x="55.54" y="9" drill="2"/>
+<hole x="80.64" y="12.01" drill="2"/>
+<hole x="55.58" y="11.96" drill="2"/>
 </plain>
 <attributes>
@@
 <wire x1="64.77" y1="40.64" x2="67.31" y2="40.64" width="0.4064" layer="16"/>
 <wire x1="76.2" y1="40.64" x2="80.01" y2="40.64" width="0.4064" layer="16"/>
+<via x="34.3" y="34.31" extent="1-16" drill="0.7" diameter="1.016" shape="square"/>
 <wire x1="75.565" y1="40.57" x2="76.2" y2="40.64" width="0" layer="19" extent="16-16"/>
 <wire x1="71.595" y1="38.77" x2="75.565" y2="40.57" width="0" layer="19" extent="16-16"/>
@@
 <via x="39.37" y="29.21" extent="1-16" drill="0.6" diameter="1.016"/>
 <wire x1="39.37" y1="29.21" x2="35.56" y2="29.21" width="0.6096" layer="16"/>
+<via x="83.82" y="29.21" extent="1-16" drill="0.7" diameter="1.016" shape="square"/>
 </signal>
 <signal name="KTIR_1">
@@
 <wire x1="19.05" y1="24.77" x2="19.05" y2="33.02" width="0.6096" layer="1"/>
 <wire x1="19.05" y1="33.02" x2="22.86" y2="33.02" width="0.6096" layer="1"/>
+<via x="22.86" y="34.29" extent="1-16" drill="0.7" diameter="1.016" shape="square"/>
+</signal>
+<signal name="N$10">
+<via x="57.19" y="22.28" extent="1-16" drill="0.7" diameter="1.016" shape="square"/>
+</signal>
+<signal name="N$11">
+<via x="57.14" y="29.24" extent="1-16" drill="0.7" diameter="1.016" shape="square"/>
+</signal>
+<signal name="N$12">
+<via x="39.38" y="29.22" extent="1-16" drill="0.7" diameter="1.016" shape="square"/>
+</signal>
+<signal name="N$14">
+<via x="22.85" y="27.01" extent="1-16" drill="0.7" diameter="1.016" shape="square"/>
+</signal>
+<signal name="N$15">
+<via x="5.11" y="27.97" extent="1-16" drill="0.7" diameter="1.016" shape="square"/>
+</signal>
+<signal name="N$16">
+<via x="72.42" y="29.23" extent="1-16" drill="0.7" diameter="1.016" shape="square"/>
+</signal>
+<signal name="N$17">
+<via x="81.25" y="38.11" extent="1-16" drill="0.7" diameter="1.016" shape="square"/>
+</signal>
+<signal name="N$18">
+<via x="101.62" y="27.3" extent="1-16" drill="0.7" diameter="1.016" shape="square"/>
+</signal>
+<signal name="N$19">
+<via x="114.21" y="19.86" extent="1-16" drill="0.7" diameter="1.016" shape="square"/>
 </signal>
 </signals>
